File: PCB_LSH20_3P_pack/PCB_LSH20_3P_pack.kicad_pcb (KiCad board)
At the start: 2 copper layers, 99 x 69 mm, 8 parts, among them J1 Conn_01x02_Pin, J2 Conn_01x02_Pin

Commit message: v1
Parts:
- BT1, BT2, BT3: moved to F.Cu
- BT4, BT5, BT6: moved to B.Cu
- moved BT1 113.1 mm to (87.0, 81.7), turned to 0 degrees
- moved BT5 83.3 mm to (117.0, 81.7), turned to 180 degrees
- moved J2 80.6 mm to (135.0, 80.7)
- moved BT2 50.9 mm to (117.0, 81.7), turned to 0 degrees
- moved BT4 47.9 mm to (87.0, 81.7), turned to 180 degrees
- moved J1 23.7 mm to (99.5, 80.7)
- moved BT6 22.7 mm to (147.0, 81.7), turned to 180 degrees
- moved BT3 17.8 mm to (147.0, 81.7), turned to 0 degrees
Routing:
- net GND: track 322.3 -> 225.6 mm, vias 21 -> 24
- net +3.3V: track 310.9 -> 226.2 mm, vias 21 -> 24
- net (no net): vias 0 -> 2
Other:
- board size 99 x 69 mm -> 72 x 59.5 mm
